File: PongSat_v3r5.sch (EAGLE design)
At the start: 33 parts, among them U1 MIC5129 3v3, U2 Micro SD, X1 USB-MICROB, Y1 8MHz

Commit message: Updated to Version 3 Revision 5
I2C header is now PTH, and various other slight tweaks have been
applied. New Gerber filed also committed. Directory structure also
simplified and reorganised.
Parts:
- I2C: device SparkFun-Connectors:M04SMD -> SparkFun-Connectors:M04PTH
Changed lines of the file:
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@@
 <part name="GND12" library="SparkFun-Aesthetics" deviceset="GND" device=""/>
 <part name="P+6" library="SparkFun-Aesthetics" deviceset="3.3V" device=""/>
-<part name="I2C" library="SparkFun-Connectors" deviceset="M04" device="SMD" value="3.3V"/>
+<part name="I2C" library="SparkFun-Connectors" deviceset="M04" device="PTH" value="3.3V"/>
 <part name="P+7" library="SparkFun-Aesthetics" deviceset="3.3V" device=""/>
 <part name="GND13" library="SparkFun-Aesthetics" deviceset="GND" device=""/>
