File: PongSat_v3r6.brd (EAGLE design)
At the start: 39 x 39 mm, 36 parts, among them U1 MIC5129 3v3, U2 Micro SD, X1 USB-MICROB, Y1 8MHz

Commit message: Minor Fixes
Routing:
- net 3.3V: track 134.6 -> 135.4 mm
Changed lines of the file:
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@@
 <setting verticaltext="up"/>
 </settings>
-<grid distance="8" unitdist="mil" unit="mil" style="dots" multiple="1" display="yes" altdistance="0.05" altunitdist="inch" altunit="inch"/>
+<grid distance="0.5" unitdist="mm" unit="mm" style="dots" multiple="1" display="yes" altdistance="0.05" altunitdist="inch" altunit="inch"/>
 <layers>
 <layer number="1" name="Top" color="4" fill="1" visible="yes" active="yes"/>
@@
 <plain>
 <circle x="19.5" y="19.5" radius="19.5" width="0.254" layer="20"/>
-<text x="6.5" y="25.5" size="1.27" layer="21">+</text>
-<text x="14" y="25.5" size="1.27" layer="21">-</text>
+<text x="5.5" y="24.5" size="3" layer="21">+</text>
+<text x="14" y="24.5" size="3" layer="21">-</text>
 <text x="23.2" y="4.5" size="0.8128" layer="22" rot="MR90">VCC</text>
 <text x="20.7" y="4.5" size="0.8128" layer="22" rot="MR90">GND</text>
@@
 <element name="U2" library="SparkFun-Connectors" package="MICRO-SD-SOCKET-PP" value="Micro SD" x="36.16" y="12.96" locked="yes" smashed="yes" rot="MR270">
 <attribute name="NAME" x="34.81" y="18.85" size="0.8128" layer="26" rot="MR270"/>
-<attribute name="VALUE" x="29.15" y="28.58" size="0.8128" layer="22" rot="MR180"/>
+<attribute name="VALUE" x="25.15" y="29.08" size="1.2" layer="22" ratio="16" rot="MR180"/>
 </element>
 <element name="I2C" library="SparkFun-Connectors" package="1X04" value="3.3V" x="23.6576" y="2.9704" locked="yes" smashed="yes" rot="MR0"/>
@@
 <wire x1="20" y1="29" x2="20.15" y2="29" width="0.254" layer="1"/>
 <wire x1="28" y1="7" x2="28" y2="7.5" width="0.254" layer="16"/>
-<wire x1="28" y1="7.5" x2="28" y2="18.5" width="0.254" layer="16"/>
+<wire x1="28" y1="7.5" x2="28" y2="8.5" width="0.254" layer="16"/>
+<wire x1="28" y1="8.5" x2="29" y2="9.5" width="0.254" layer="16"/>
+<wire x1="29" y1="9.5" x2="29" y2="11" width="0.254" layer="16"/>
+<wire x1="29" y1="11" x2="28" y2="12" width="0.254" layer="16"/>
+<wire x1="28" y1="12" x2="28" y2="18.5" width="0.254" layer="16"/>
 <wire x1="8.5" y1="13.5" x2="8" y2="13" width="0.254" layer="1"/>
 <wire x1="8" y1="13" x2="8" y2="9" width="0.254" layer="1"/>
